File: 4 digit VA module.kicad_sch (KiCad schematic)
At the start: 55 parts, among them J1 Conn_01x02, J2 Conn_01x02, J3 Conn_01x02, J4 Conn_01x03_Pin, J5 Conn_01x02_Socket, J6 Conn_01x02_Socket, Q1 BC817, Q2 BC817, Q3 BC817, Q4 BC817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

Commit message: Samo 7 seg je kinezijum
12 bit je malo cheapout, ukupna cena 5.8 EUR.
Parts:
- removed U3, U4: CC56-12GWA, Display_7Segment:CC56-12GWA, symbol Display_Character:CC56-12GWA
- added J7: Conn_01x02_Socket, Connector_PinHeader_2.54mm:PinHeader_1x02_P2.54mm_Vertical, symbol Connector:Conn_01x02_Socket
- added U3, U4: 3641BS, Pretty feet:3641, symbol SPICE_diodes:3641BS
- U2: Price 1.94 -> 1.3
Connections:
- net V_IN_MUX: now also U5.21 (PB10)
- net at R29.1: now also U3.3 (DPX)
- net at R26.1: now also U3.1 (e)
- net at R27.1: now also U3.10 (f)
- net at R22.1: now also U3.11 (a)
- net at Q4.3 (C): now also U3.12 (CC1)
- net at R25.1: now also U3.2 (d)
- net at R24.1: now also U3.4 (c)
- net at R28.1: now also U3.5 (g)
- net at Q1.3 (C): now also U3.6 (CC4)
- net at R23.1: now also U3.7 (b)
- net at Q2.3 (C): now also U3.8 (CC3)
- net at Q3.3 (C): now also U3.9 (CC2)
- net at R10.1: now also U4.11 (a)
- net at R20.1: now also U4.5 (g)
- net at R16.1: now also U4.1 (e)
- net CAL: now reaches U5.1 (PC0)
- net CAL: now also J7.1 (Pin_1)
- net STATE: now reaches U5.2 (PC13)
- net STATE: now also J7.2 (Pin_2)
- net at Q8.3 (C): now also U4.12 (CC1)
- net at Q6.3 (C): now also U4.8 (CC3)
- net at R19.1: now also U4.10 (f)
- net at R14.1: now also U4.2 (d)
- net at R21.1: now also U4.3 (DPX)
- net at R12.1: now also U4.4 (c)
- net at Q5.3 (C): now also U4.6 (CC4)
- net at R11.1: now also U4.7 (b)
- net at Q7.3 (C): now also U4.9 (CC2)
Other:
- note added: "12 bit sa oversample-ingom bi trebao da bude dovoljno dobar"
- note added: "možda je glupo da se koriste svi ovi tranzistori"

Commit message: Work in progress
Parts:
- removed J2, J3: Conn_01x02, TerminalBlock:TerminalBlock_Altech_AK300-2_P5.00mm, symbol Connector_Generic:Conn_01x02
- removed U6: SN74LV4052, Package_SO:SOIC-16_3.9x9.9mm_P1.27mm, symbol SPICE_Analog_Switch:SN74LV4052
- added J2: Conn_01x03, Connector_JST:JST_EH_B3B-EH-A_1x03_P2.50mm_Vertical, symbol Connector_Generic:Conn_01x03
- added U8: 74LVC1G3157, Package_TO_SOT_SMD:SOT-363_SC-70-6_Handsoldering, symbol 74xGxx:74LVC1G3157
- U2: Price 1.3 -> 1.63
Connections:
- net 0: now also J2.1 (Pin_1), U8.2 (GND)
- net 3.3V: now also U8.5 (VCC)
- net I_OUT: now also U8.1
- net PSU: now also J2.2 (Pin_2)
- net VA_SEL: now also U8.6
- net V_IN_MUX: no longer U7.3 (+)
- net V_in_pos: now also J2.3 (Pin_3)
- net at U2.3 (IN+): now also U8.4
- net at U7.2 (-), U7.6: now also U8.3
- net LEVEL_JUDGE: no longer names the net of R15.1, R17.2
- net LEVEL_JUDGE: now also U7.3 (+); no longer U5.10 (PA0)
Other:
- moved on the sheet: U7

Commit message: BOM za ne kinezijum je 5.3, totalno prihvatljivo.
Parts:
- removed C1: 100n, Capacitor_SMD:C_1206_3216Metric_Pad1.33x1.80mm_HandSolder, symbol Device:C
- removed J4: Conn_01x03_Pin, Connector_PinHeader_2.54mm:PinHeader_1x03_P2.54mm_Vertical, symbol Connector:Conn_01x03_Pin
- removed J5, J6, J7: Conn_01x02_Socket, Connector_PinHeader_2.54mm:PinHeader_1x02_P2.54mm_Vertical, symbol Connector:Conn_01x02_Socket
- removed R10, R11, R12, R14, R16, R19, R20, R21, R22, R23, R24, R25, R26, R27, R28, R29: 220, Resistor_SMD:R_1206_3216Metric_Pad1.30x1.75mm_HandSolder, symbol Device:R
- removed R15: 24.9k, Resistor_SMD:R_1206_3216Metric_Pad1.30x1.75mm_HandSolder, symbol Device:R
- removed R17: 220k, Resistor_SMD:R_1206_3216Metric_Pad1.30x1.75mm_HandSolder, symbol Device:R
- removed R30: 4.99k, Resistor_SMD:R_1206_3216Metric_Pad1.30x1.75mm_HandSolder, symbol Device:R
- removed U3, U4: 3641BS, Pretty feet:3641, symbol SPICE_diodes:3641BS
- removed U5: STM32L010C6Tx, Package_QFP:LQFP-48_7x7mm_P0.5mm, symbol MCU_ST_STM32L0:STM32L010C6Tx
- removed U7: TLV07, Package_SO:SOIC-8_3.9x4.9mm_P1.27mm, symbol SPICE_opamps:TLV07
- added C2, C3, C4, C5, C6: 100n, Capacitor_SMD:C_1206_3216Metric_Pad1.33x1.80mm_HandSolder, symbol Device:C
- added J10, J3: Conn_01x02_Socket, Connector_PinHeader_2.54mm:PinHeader_1x02_P2.54mm_Vertical, symbol Connector:Conn_01x02_Socket
- added J8, J9: Conn_01x03_Pin, Connector_PinHeader_2.54mm:PinHeader_1x03_P2.54mm_Vertical, symbol Connector:Conn_01x03_Pin
- added R32, R33, R34, R35, R36, R37, R38, R39: 220, Resistor_SMD:R_0603_1608Metric_Pad0.98x0.95mm_HandSolder, symbol Device:R
- added U3, U4: 2841BS, Pretty feet:2841, symbol SPICE_diodes:2841BS
- added U5: LM321, Package_TO_SOT_SMD:SOT-23-5, symbol SPICE_opamps:LM321
- added U6: STM32L010C6Tx, Package_QFP:LQFP-48_7x7mm_P0.5mm, symbol MCU_ST_STM32L0:STM32L010C6Tx
- Q1, Q2, Q3, Q4, Q5, Q6, Q7, Q8: Price 0.05 -> 0.022
- R1: value 50m -> 10m; Price 0.38 -> 0.245
- R13, R2, R3, R4, R5, R6, R7, R8, R9: footprint Resistor_SMD:R_1206_3216Metric_Pad1.30x1.75mm_HandSolder -> Resistor_SMD:R_0603_1608Metric_Pad0.98x0.95mm_HandSolder
- R18: value 750k -> 1Meg; footprint Resistor_SMD:R_1206_3216Metric_Pad1.30x1.75mm_HandSolder -> Resistor_SMD:R_0603_1608Metric_Pad0.98x0.95mm_HandSolder
- R31: value 100 -> 25.64k; footprint Resistor_SMD:R_1206_3216Metric_Pad1.30x1.75mm_HandSolder -> Resistor_SMD:R_0603_1608Metric_Pad0.98x0.95mm_HandSolder
Connections:
- net 0: now also C2.1, C3.1, C4.1, C5.1, C6.1, J8.3 (Pin_3), J9.1 (Pin_1), U5.2 (V-), U6.23 (VSS), U6.35 (VSS), U6.47 (VSS), U6.8 (VSSA)
- net 3.3V: now also C3.2, C4.2, C5.2, C6.2, J8.1 (Pin_1), U5.5 (V+), U6.24 (VDD), U6.36 (VDD), U6.48 (VDD), U6.9 (VDDA)
- net A: now also R35.2, U3.11 (a), U4.11 (a)
- net B: now also R38.1, U3.7 (b), U4.7 (b)
- net C: now also R36.2, U3.4 (c), U4.4 (c)
- net CAL: now also J3.1 (Pin_1), U6.1 (PC0)
- net CC1: now also U6.39 (PB3)
- net CC2: now also U6.40 (PB4)
- net CC3: now also U6.41 (PB5)
- net CC4: now also U6.46 (PB9)
- net CC5: now also U6.18 (PB0)
- net CC6: now also U6.19 (PB1)
- net CC7: now also U6.20 (PB2)
- net CC8: now also U6.21 (PB10)
- net CNV_START: now also U6.14 (PA4)
- net D: now also R33.2, U3.2 (d), U4.2 (d)
- net DP: now also R39.1, U3.3 (DPX), U4.3 (DPX)
- net E: now also R32.1, U3.1 (e), U4.1 (e)
- net F: now also R34.2, U3.10 (f), U4.10 (f)
- net G: now also R37.1, U3.5 (g), U4.5 (g)
- net SPI_CLK: now also U6.15 (PA5)
- net SPI_MISO: now also U6.16 (PA6)
- net SPI_MOSI: now also U6.17 (PA7)
- net STATE: now also J3.2 (Pin_2), U6.2 (PC13)
- net SWCLK: now also J9.2 (Pin_2), U6.37 (PA14)
- net SWDIO: now also J9.3 (Pin_3), U6.34 (PA13)
- net USART_RX: now also J10.2 (Pin_2), U6.13 (PA3)
- net USART_TX: now also J10.1 (Pin_1), U6.12 (PA2)
- net VA_SEL: now also U6.42 (PB6)
- net V_IN_MUX: now also U6.45 (PB8)
- net V_RANGE: now also U6.43 (PB7)
- net at R18.2: now also R31.1, U5.1 (+)
- net at U8.3: now also U5.3 (-), U5.4
- net at Q8.3 (C): now also U3.12 (CC1)
- net at Q2.3 (C): now also U4.8 (CC3)
- net at Q6.3 (C): now also U3.8 (CC3)
- net at Q3.3 (C): now also U4.9 (CC2)
- net at Q1.3 (C): now also U4.6 (CC4)
- net at Q7.3 (C): now also U3.9 (CC2)
- net at Q4.3 (C): now also U4.12 (CC1)
- net at Q5.3 (C): now also U3.6 (CC4)
- new net: R39.2, U6.29 (PA8)
- new net: C2.2, U6.7 (NRST)
- new net: R34.1, U6.25 (PB12)
- new net: R33.1, U6.22 (PB11)
- new net: R32.2, U6.27 (PB14)
- new net: R36.1, U6.30 (PA9)
- new net: R37.2, U6.31 (PA10)
- new net: R38.2, U6.32 (PA11)
- new net: R35.1, U6.33 (PA12)
- new net: J8.2 (Pin_2), U6.44 (BOOT0)
Other:
- moved on the sheet: R18, R31, U8B

Commit message: WIP
Parts:
- removed J10: Conn_01x02_Socket, Connector_PinHeader_2.54mm:PinHeader_1x02_P2.54mm_Vertical, symbol Connector:Conn_01x02_Socket
- removed J8: Conn_01x03_Pin, Connector_PinHeader_2.54mm:PinHeader_1x03_P2.54mm_Vertical, symbol Connector:Conn_01x03_Pin
- removed U10: AP2112K-3.3, Package_TO_SOT_SMD:SOT-23-5, symbol Regulator_Linear:AP2112K-3.3
- added C1, C7, C8: 1u, Capacitor_SMD:C_0603_1608Metric_Pad1.08x0.95mm_HandSolder, symbol Device:C
- added C9: 100p, Capacitor_SMD:C_0603_1608Metric_Pad1.08x0.95mm_HandSolder, symbol Device:C
- added U7: AP2210K-3.3TRG1, Package_TO_SOT_SMD:SOT-23-5, symbol SPICE_voltage_references:AP2210K-3.3TRG1
- C2, C3, C4, C5, C6: footprint Capacitor_SMD:C_1206_3216Metric_Pad1.33x1.80mm_HandSolder -> Capacitor_SMD:C_0603_1608Metric_Pad1.08x0.95mm_HandSolder
- R13: value 900k -> 1k
Connections:
- net 0: now also C1.2, C7.2, C8.2, C9.2, U7.2 (GND)
- net 3.3V: now also C7.1, C8.1, U7.3 (EN), U7.5 (OUT)
- net CC1: now also R9.2; no longer R5.2
- net CC2: now also R8.2; no longer R2.2
- net CC3: now also R7.2; no longer R3.2
- net CC4: now also R6.2, U6.42 (PB6); no longer R4.2, U6.46 (PB9)
- net CC5: now also R5.2; no longer R9.2
- net CC6: now also R2.2; no longer R8.2
- net CC7: now also R3.2; no longer R7.2
- net CC8: now also R4.2; no longer R6.2
- net PSU: now also C1.1, U7.1 (IN)
- net SWCLK: now also J9.3 (Pin_3); no longer J9.2 (Pin_2)
- net SWDIO: now also J9.2 (Pin_2); no longer J9.3 (Pin_3)
- net VA_SEL: now also U6.46 (PB9); no longer U6.42 (PB6)
- net USART_RX: no longer names the net of U6.13 (PA3)
- net USART_TX: no longer names the net of U6.12 (PA2)
- new net: C9.1, U7.4 (BP)
Other:
- note added: "14 bit + oversampling je vrv dosta"
- note added: "2.5V range sa 14 bit i INL od 0.27 pravi grešku od 41.2 uV, pa kad se skalira na 100V, greška je 1.6 mV. Totalno prihvatljivo"
- note added: "za 1 mA, 0.8V razlike tkd 800 ili 1 kOhm"
- note removed: "12 bit sa oversample-ingom bi trebao da bude dovoljno dobar"
- moved on the sheet: J2, U2, U5, U8B

Commit message: Izgleda kao da je PCB gotov, treba proveriti dimenziju.
Parts:
- added C10, C11, C12: 100n, Capacitor_SMD:C_0603_1608Metric_Pad1.08x0.95mm_HandSolder, symbol Device:C
Connections:
- net 0: now also C10.1, C11.1, C12.1
- net 3.3V: now also C10.2, C11.2, C12.2
Other:
- note added: "PROVERI DIMENZIJE"
- note removed: "Možda treba clock kristal"
